Commit message: Fixed broken JointPositionControllers for ur5e_gripper_gazebo

File: src/ur5e_gripper/ur5e_gripper_description/urdf/hand_e.xacro (robot description, xacro)
@@ -2,5 +2,7 @@
 <robot name="robotiq_hande_gripper" xmlns:xacro="http://wiki.ros.org/xacro">
     <xacro:include filename="$(find robotiq_description)/urdf/robotiq_hande_gripper.urdf.xacro" />
-    <xacro:robotiq_hande_gripper prefix="" parent="tool0">
+    <xacro:robotiq_hande_gripper
+        prefix=""
+        parent="tool0">
         <origin xyz="0 0 0" rpy="0 0 0" />
     </xacro:robotiq_hande_gripper>

File: src/ur5e_gripper/ur5e_gripper_gazebo/urdf/ur_macro.xacro (robot description, xacro)
@@ -31,5 +31,6 @@
   -->
   <!-- Definition of the main macro -->
-  <xacro:macro name="ur_robot_gazebo" params="
+  <xacro:macro name="ur_robot_gazebo"
+    params="
    prefix
    joint_limits_parameters_file
@@ -46,5 +47,5 @@
       the definitions for the real robot.
     -->
-  <xacro:include filename="$(find ur_description)/urdf/inc/ur_macro.xacro"/>
+    <xacro:include filename="$(find ur_description)/urdf/inc/ur_macro.xacro" />
     <!-- Instantiate model for the REAL robot. -->
     <xacro:ur_robot

Commit message: Edited ur5e_gripper_description/gazebo configurations

File: src/ur5e_gripper/ur5e_gripper_description/urdf/hand_e.xacro (robot description, xacro)
@@ -5,5 +5,5 @@
         prefix=""
         parent="tool0">
-        <origin xyz="0 0 0" rpy="0 0 0" />
+        <origin xyz="0 0 0" rpy="0 0 1.57" />
     </xacro:robotiq_hande_gripper>
 </robot>
