Commit message: Rotated tool in ur5 gripper urdf

File: src/ur5e_gripper/ur5e_gripper_description/urdf/ur_hand_e.xacro (robot description, xacro)
@@ -24,5 +24,5 @@
             prefix="${prefix}"
             parent="${prefix}tool0">
-            <origin xyz="0 0 0" rpy="0 0 1.57" />
+            <origin xyz="0 0 0" rpy="0 0 0" />
         </xacro:robotiq_hande_gripper>
     </xacro:macro>
