Commit message: Better use of xacro macros in ur+gripper description files, added joint limits config file

File: src/ur5e_gripper/ur5e_gripper_description/urdf/ur5e_gripper_hand_e.xacro (robot description, xacro)
@@ -2,5 +2,5 @@
 <robot name="ur5e_gripper" xmlns:xacro="http://wiki.ros.org/xacro">
     <xacro:include filename="$(find ur_description)/urdf/inc/ur_macro.xacro" />
-    <xacro:include filename="$(find ur5e_gripper_description)/urdf/hand_e.xacro" />
+    <xacro:include filename="$(find ur5e_gripper_description)/urdf/hande_macro.xacro" />
     <!-- parameters -->
     <xacro:arg name="joint_limit_params" default="" />
@@ -16,11 +16,10 @@
     <xacro:arg name="safety_pos_margin" default="0.15" />
     <xacro:arg name="safety_k_position" default="20" />
-    <!-- arm -->
-    <xacro:ur_robot
+    <xacro:ur5_hand_e
         prefix=""
-        joint_limits_parameters_file="$(arg joint_limit_params)"
-        kinematics_parameters_file="$(arg kinematics_params)"
-        physical_parameters_file="$(arg physical_params)"
-        visual_parameters_file="$(arg visual_params)"
+        joint_limit_params="$(arg joint_limit_params)"
+        kinematics_params="$(arg kinematics_params)"
+        physical_params="$(arg physical_params)"
+        visual_params="$(arg visual_params)"
         transmission_hw_interface="$(arg transmission_hw_interface)"
         safety_limits="$(arg safety_limits)"

File: src/ur5e_gripper/ur5e_gripper_description/urdf/ur_hand_e.xacro (robot description, xacro)
@@ -21,9 +21,7 @@
             safety_pos_margin="${safety_pos_margin}"
             safety_k_position="${safety_k_position}" />
-        <xacro:robotiq_hande_gripper
-            prefix="${prefix}"
-            parent="${prefix}tool0">
-            <origin xyz="0 0 0" rpy="0 0 0" />
-        </xacro:robotiq_hande_gripper>
+        <xacro:hande_gripper
+            prefix=""
+            parent="tool0"/>
     </xacro:macro>
 </robot>

File: src/ur5e_gripper/ur5e_gripper_gazebo/urdf/ur5e_gripper_hand_e.xacro (robot description, xacro)
@@ -2,5 +2,5 @@
 <robot name="ur5e_gripper" xmlns:xacro="http://wiki.ros.org/xacro">
     <xacro:include filename="$(find ur5e_gripper_gazebo)/urdf/ur_macro.xacro" />
-    <xacro:include filename="$(find ur5e_gripper_description)/urdf/hand_e.xacro" />
+    <xacro:include filename="$(find ur5e_gripper_description)/urdf/hande_macro.xacro" />
     <!-- parameters -->
     <xacro:arg name="joint_limit_params" default="" />
@@ -27,4 +27,7 @@
         safety_pos_margin="$(arg safety_pos_margin)"
         safety_k_position="$(arg safety_k_position)" />
+    <xacro:hande_gripper
+        prefix=""
+        parent="tool0"/>
     <link name="world" />
     <joint name="world_joint" type="fixed">
