Commit message: Fixed missing prefix in hande_macro.xacro

File: src/ur5e_gripper/ur5e_gripper_description/urdf/hande_macro.xacro (robot description, xacro)
@@ -9,6 +9,6 @@
             <origin xyz="0 0 0" rpy="0 0 0" />
         </xacro:robotiq_hande_gripper>
-        <link name="ee_link" />
-        <joint name="ee_link_joint" type="fixed">
+        <link name="${prefix}ee_link" />
+        <joint name="${prefix}ee_link_joint" type="fixed">
             <origin
                 xyz="0 0 ${z_offset}"
